File: schematics/dodohand_PCB/dodohand_PCB.sch (KiCad schematic (older format))
At the start: 19 parts, among them U1 TEENSY_LC

Commit message: add sr0_LED_shiftRegs.ino, LED_shiftRegs, LED_shiftRegs
Connections:
- net row_left/CS: now also U1.21 (15); no longer U1.20 (14)
- net row_right/CS: now also U1.25 (19); no longer U1.21 (15)
Changed lines of the file:
@@
 NoConn ~ 2050 4100
 NoConn ~ 2500 4100
-NoConn ~ 2650 4100
+NoConn ~ 3400 4100
 NoConn ~ 2800 4100
 NoConn ~ 3800 4650
@@
 	8250 1900 8250 3800
 Wire Wire Line
-	3250 2100 8050 2100
-Wire Wire Line
-	3250 4100 3250 2100
+	2650 2100 8050 2100
+Wire Wire Line
+	2650 4100 2650 2100
 Connection ~ 5550 3350
 Connection ~ 5750 3150
@@
 	3550 5750 5050 5750
 Wire Wire Line
-	3400 2350 6350 2350
-Wire Wire Line
-	3400 4100 3400 2350
+	3250 2350 6350 2350
+Wire Wire Line
+	3250 4100 3250 2350
 Wire Wire Line
 	5950 2950 5950 3800
@@
 Wire Wire Line
 	5550 3350 5550 3800
-Wire Wire Line
-	3100 4100 4350 4100
 Wire Wire Line
 	2500 5750 2500 6000
@@
 	4000 4400 4200 4400
 Wire Wire Line
-	4350 4100 4350 4400
+	4350 4050 4350 4400
 Wire Wire Line
 	4500 3850 4500 4400
@@
 Connection ~ 4500 5250
 Connection ~ 4350 5250
+Wire Wire Line
+	4350 4050 3100 4050
+Wire Wire Line
+	3100 4050 3100 4100
 $EndSCHEMATC
