File: examples/shiftRegs/sr4_keys/schematics/dodohand_BB.sch (KiCad schematic (older format))
At the start: 1 part, among them U1 TEENSY_LC

Commit message: updated dodoHand shift-register schematics
Parts:
- added 0.1uF1: C, symbol C
- added C1, C2: 0.1uF, symbol C
- added D1, D2: LED, symbol LED
- added R1, R2, R3, R4, R6, R7: 4.7k, symbol R
- added R5: 470, symbol R
- added SW1, SW2: SW_PUSH_SMALL_H, symbol SW_PUSH_SMALL_H
- added U2, U4: 74AHC1G126, symbol 74AHC1G126
- added U3, U5: 74HC165., symbol 74HC165.
- added U6: 74HC595, symbol 74HC595-RESCUE-dodohand_PCB
- added X1: 2keys, symbol 2keys
Connections:
- net labels removed: +3.3V, GND
- wire segments 31 -> 116
- no-connect marks 25 -> 34
