File: examples/shiftRegs/sr5_dodohand_PCB/schematics/dodohand_PCB.sch (KiCad schematic (older format))
At the start: 19 parts, among them U1 TEENSY_LC

Commit message: updated dodoHand shift-register schematics
Parts:
- removed C?: C, symbol C
- added 0.1uF1: C_Small, symbol C_Small
- added U2, U3, U4, U9: strobe_buffer, symbol strobe_buffer
- U10: renamed from U?; symbol 74HC595 -> 74HC595-RESCUE-dodohand_PCB
- gave numbers to parts that had none: 16
Connections:
- net labels removed: +3.3V, +5V, GND
- wire segments 71 -> 94
- no-connect marks 25 -> 27
Other:
- moved on the sheet: D1, D2, D3, D4, D5, D6, D7, D8, R1, R2, R3, R4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
