File: examples/shiftRegs/sr5_dodohand_PCB/kicad_schematics/dodohand_PCB.sch (KiCad schematic (older format))
At the start: 23 parts, among them U1 TEENSY_LC, U10 74HC595, U2 strobe_buffer, U3 strobe_buffer, U4 strobe_buffer, U9 strobe_buffer

Commit message: document
Connections:
- net row_left/CS renamed row_left/SS
- net row_right/CS renamed row_right/SS
Changed lines of the file:
@@
 F3 "3.3V" I T 9150 5950 60
 F4 "CLK" I T 9350 5950 60
-F5 "CS" I T 9750 5950 60
+F5 "SS" I T 9750 5950 60
 F6 "MISO" I T 9550 5950 60
 F7 "strobe" I T 9950 5950 60
@@
 F3 "3.3V" I T 10850 5950 60
 F4 "CLK" I T 11050 5950 60
-F5 "CS" I T 11450 5950 60
+F5 "SS" I T 11450 5950 60
 F6 "MISO" I T 11250 5950 60
 F7 "strobe" I T 11650 5950 60
@@
 	5850 7950 5850 8250
 Wire Wire Line
-	1750 8250 5850 8250
-Wire Wire Line
-	1750 6750 1750 8250
+	5850 8250 1750 8250
+Wire Wire Line
+	1750 8250 1750 6750
 Wire Wire Line
 	1750 6750 2300 6750
