File: examples/shiftRegs/sr5_dodohand_PCB/kicad_schematics/row.sch (KiCad schematic (older format))
At the start: 2 parts, among them U11 74AHC1G126

Commit message: document
Connections:
- net CS renamed SS
Changed lines of the file:
@@
 GND
 Text HLabel 4200 1300 1    60   Input ~ 0
-CS
+SS
 Text HLabel 4100 1300 1    60   Input ~ 0
 CLK
@@
 AR Path="/5809DAC4/580B7854" Ref="C2"  Part="1"
 AR Path="/580AEA89/580B7854" Ref="C4"  Part="1"
-F 0 "C4" V 3348 1750 50  0000 C CNN
+F 0 "C2" V 3348 1750 50  0000 C CNN
 F 1 "C" V 3439 1750 50  0000 C CNN
 F 2 "" H 3638 1600 50  0000 C CNN
@@
 F6 "3.3V" I T 10200 5400 60
 F7 "CLK" I T 10350 5400 60
-F8 "CS" I T 10450 5400 60
+F8 "SS" I T 10450 5400 60
 $EndSheet
 Wire Wire Line
@@
 F6 "3.3V" I T 6000 5400 60
 F7 "CLK" I T 6150 5400 60
-F8 "CS" I T 6250 5400 60
+F8 "SS" I T 6250 5400 60
 $EndSheet
 Wire Wire Line
@@
 F6 "3.3V" I T 8200 5400 60
 F7 "CLK" I T 8350 5400 60
-F8 "CS" I T 8450 5400 60
+F8 "SS" I T 8450 5400 60
 $EndSheet
 $Sheet
@@
 F3 "GND" I T 3300 5400 60
 F4 "HQ" I T 3750 5400 60
-F5 "SER" I T 3550 5400 60
-F6 "3.3V" I T 3950 5400 60
-F7 "CLK" I T 4100 5400 60
-F8 "CS" I T 4200 5400 60
+F5 "3.3V" I T 3950 5400 60
+F6 "CLK" I T 4100 5400 60
+F7 "SS" I T 4200 5400 60
 $EndSheet
 Wire Wire Line
@@
 AR Path="/5809DAC4/582FA7A2" Ref="U11"  Part="1"
 AR Path="/580AEA89/582FA7A2" Ref="U16"  Part="1"
-F 0 "U16" V 5196 2222 50  0000 R CNN
+F 0 "U11" V 5196 2222 50  0000 R CNN
 F 1 "74AHC1G126" V 5105 2222 50  0000 R CNN
 F 2 "" H 5000 2200 50  0000 C CNN
