File: examples/shiftRegs/sr5_dodohand_PCB/kicad_schematics/shiftReg_2keys.sch (KiCad schematic (older format))
At the start: 3 parts, among them U5 74HC165, X4 2buttons

Commit message: document
Connections:
- net CS renamed SS
- net SER: no longer names the net of U5.10 (SER)
- no-connect marks 1 -> 2
Changed lines of the file:
@@
 GND
 Text HLabel 6400 1000 1    60   Input ~ 0
-CS
+SS
 Text HLabel 6300 1100 1    60   Input ~ 0
 CLK
@@
 AR Path="/580AEA89/580F922E/5809DC59" Ref="U14"  Part="1"
 AR Path="/580AEA89/580FCD1C/5809DC59" Ref="U15"  Part="1"
-F 0 "U15" V 5904 2928 50  0000 L CNN
+F 0 "U8" V 5904 2928 50  0000 L CNN
 F 1 "74HC165" V 5995 2928 50  0000 L CNN
 F 2 "" H 5950 2350 50  0000 C CNN
@@
 AR Path="/580AEA89/580F922E/580C1CC7" Ref="X28"  Part="1"
 AR Path="/580AEA89/580FCD1C/580C1CC7" Ref="X32"  Part="1"
-F 0 "X32" V 7553 4822 60  0000 R CNN
+F 0 "X16" V 7553 4822 60  0000 R CNN
 F 1 "2buttons" V 7447 4822 60  0000 R CNN
 F 2 "" H 7550 5100 60  0000 C CNN
@@
 AR Path="/580AEA89/580F922E/580C3691" Ref="RA14"  Part="1"
 AR Path="/580AEA89/580FCD1C/580C3691" Ref="RA16"  Part="1"
-F 0 "RA16" H 6428 3703 60  0000 L CNN
+F 0 "RA8" H 6428 3703 60  0000 L CNN
 F 1 "resistor_array" H 6428 3597 60  0000 L CNN
 F 2 "" H 6200 3650 60  0001 C CNN
@@
 HQ
 Wire Wire Line
-	5850 1650 5850 1000
-Text HLabel 5850 1000 1    60   Input ~ 0
-SER
-Wire Wire Line
 	8250 6350 8250 1100
 Wire Wire Line
@@
 Wire Wire Line
 	5550 3050 5550 3950
+NoConn ~ 5850 1650
 $EndSCHEMATC
