File: examples/shiftRegs/sr5_dodohand_PCB/kicad_schematics/shiftReg_8keys.sch (KiCad schematic (older format))
At the start: 7 parts, among them U5 74HC165, X1 2keys, X2 2keys, X3 2keys, X4 2keys

Commit message: document
Connections:
- net CS renamed SS
Changed lines of the file:
@@
 $Descr A4 11693 8268
 encoding utf-8
-Sheet 3 11
+Sheet 5 11
 Title "8 shift registers and 8 keys"
 Date ""
@@
 GND
 Text HLabel 6400 1000 1    60   Input ~ 0
-CS
+SS
 Text HLabel 6300 1100 1    60   Input ~ 0
 CLK
@@
 AR Path="/580AEA89/580F922E/580B3CEE" Ref="X26"  Part="1"
 AR Path="/580AEA89/580FCD1C/580B3CEE" Ref="X30"  Part="1"
-F 0 "X26" V 5403 4822 60  0000 R CNN
+F 0 "X10" V 5403 4822 60  0000 R CNN
 F 1 "2keys" V 5297 4822 60  0000 R CNN
 F 2 "" H 5400 5100 60  0000 C CNN
@@
 AR Path="/580AEA89/580F922E/580AE437" Ref="RA13"  Part="1"
 AR Path="/580AEA89/580FCD1C/580AE437" Ref="RA15"  Part="1"
-F 0 "RA13" H 5928 3703 60  0000 L CNN
+F 0 "RA5" H 5928 3703 60  0000 L CNN
 F 1 "resistor_array" H 5928 3597 60  0000 L CNN
 F 2 "" H 5700 3650 60  0001 C CNN
@@
 AR Path="/580AEA89/580F922E/580D709A" Ref="U14"  Part="1"
 AR Path="/580AEA89/580FCD1C/580D709A" Ref="U15"  Part="1"
-F 0 "U14" V 5904 2928 50  0000 L CNN
+F 0 "U7" V 5904 2928 50  0000 L CNN
 F 1 "74HC165" V 5995 2928 50  0000 L CNN
 F 2 "" H 5950 2350 50  0000 C CNN
@@
 AR Path="/580AEA89/580F922E/580B560C" Ref="X25"  Part="1"
 AR Path="/580AEA89/580FCD1C/580B560C" Ref="X29"  Part="1"
-F 0 "X25" V 4653 4822 60  0000 R CNN
+F 0 "X9" V 4653 4822 60  0000 R CNN
 F 1 "2keys" V 4547 4822 60  0000 R CNN
 F 2 "" H 4650 5100 60  0000 C CNN
@@
 AR Path="/580AEA89/580F922E/580C13B3" Ref="X27"  Part="1"
 AR Path="/580AEA89/580FCD1C/580C13B3" Ref="X31"  Part="1"
-F 0 "X27" V 6803 4822 60  0000 R CNN
+F 0 "X11" V 6803 4822 60  0000 R CNN
 F 1 "2keys" V 6697 4822 60  0000 R CNN
 F 2 "" H 6800 5100 60  0000 C CNN
@@
 AR Path="/580AEA89/580F922E/580D709B" Ref="X28"  Part="1"
 AR Path="/580AEA89/580FCD1C/580D709B" Ref="X32"  Part="1"
-F 0 "X28" V 7553 4822 60  0000 R CNN
+F 0 "X12" V 7553 4822 60  0000 R CNN
 F 1 "2keys" V 7447 4822 60  0000 R CNN
 F 2 "" H 7550 5100 60  0000 C CNN
@@
 AR Path="/580AEA89/580F922E/580D709C" Ref="RA14"  Part="1"
 AR Path="/580AEA89/580FCD1C/580D709C" Ref="RA16"  Part="1"
-F 0 "RA14" H 6428 3703 60  0000 L CNN
+F 0 "RA6" H 6428 3703 60  0000 L CNN
 F 1 "resistor_array" H 6428 3597 60  0000 L CNN
 F 2 "" H 6200 3650 60  0001 C CNN
